File: Autobalancer Module/PID.kicad_sch (KiCad schematic)
At the start: 56 parts, among them U19 SGM4157YC6, U22 EinsPID, U24 LTC2633, U25 SGM4157YC6, U26 SGM4157YC6, U27 SGM4157YC6, U28 LTC2633

Commit message: Add files via upload
Parts:
- R87, R88: value 10k -> 220; LCSC C25744 -> C25091
Changed lines of the file:
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@@
     (in_bom yes) (on_board yes)
     (property "Reference" "R88" (id 0) (at 119.4816 29.845 90))
-    (property "Value" "10k" (id 1) (at 121.793 29.845 90))
+    (property "Value" "220" (id 1) (at 121.793 29.845 90))
     (property "Footprint" "Resistor_SMD:R_0402_1005Metric" (id 2) (at 124.46 29.845 0)
       (effects (font (size 1.27 1.27)) hide)
@@
       (effects (font (size 1.27 1.27)) hide)
     )
-    (property "LCSC" "C25744" (id 4) (at 124.46 29.845 90)
+    (property "LCSC" "C25091" (id 4) (at 124.46 29.845 90)
       (effects (font (size 1.27 1.27)) hide)
     )
@@
     (in_bom yes) (on_board yes)
     (property "Reference" "R87" (id 0) (at 119.4816 57.785 90))
-    (property "Value" "10k" (id 1) (at 121.793 57.785 90))
+    (property "Value" "220" (id 1) (at 121.793 57.785 90))
     (property "Footprint" "Resistor_SMD:R_0402_1005Metric" (id 2) (at 124.46 57.785 0)
       (effects (font (size 1.27 1.27)) hide)
@@
       (effects (font (size 1.27 1.27)) hide)
     )
-    (property "LCSC" "C25744" (id 4) (at 124.46 57.785 90)
-      (effects (font (size 1.27 1.27)) hide)
-    )
+    (property "LCSC" "C25091" (id 4) (at 124.46 57.785 90)
+      (effects (font (size 1.27 1.27)) hide)
+    )
